Commit message: Added repo latest release

File: dbw_mkz_ros/dbw_mkz_description/urdf/mkz.urdf.xacro (robot description, xacro)
@@ -1,93 +1,4 @@
 <?xml version="1.0"?>
-<robot name="mobility_base" xmlns:xacro="http://www.ros.org/wiki/xacro" >
-  <xacro:property name="M_PI" value="3.1415926535897931" />
-  <xacro:property name="wheel_base_x" value="${2.8448}" />
-  <xacro:property name="wheel_base_y" value="${1.5748/2}" />
-  <xacro:property name="wheel_radius" value="0.2413" />
-  <!-- Materials -->
-  <xacro:macro name="darkred_material" >
-    <material name="darkred" >
-      <color rgba=".5 .1 .1 1"/>
-    </material>
-  </xacro:macro>
-  <xacro:macro name="grey_material" >
-    <material name="grey" >
-      <color rgba=".5 .5 .5 1"/>
-    </material>
-  </xacro:macro>
-  <xacro:macro name="black_material" >
-    <material name="black" >
-      <color rgba=".1 .1 .1 1"/>
-    </material>
-  </xacro:macro>
-  <xacro:macro name="steering" params="suffix reflecty" >
-    <link name="steer${suffix}" >
-      <inertial>
-        <mass value="1" />
-        <inertia ixx="1.0" ixy="0.0" ixz="0.0"
-          iyx="0.0" iyy="1.0" iyz="0.0"
-          izx="0.0" izy="0.0" izz="1.0" />
-      </inertial>
-    </link>
-    <joint name="steer${suffix}" type="continuous" >
-      <parent link="base_link" />
-      <child link="steer${suffix}" />
-      <origin xyz="${wheel_base_x} ${reflecty*wheel_base_y} 0" rpy="0 0 0" />
-      <axis xyz="0 0 1" />
-    </joint>
-  </xacro:macro>
-  <xacro:macro name="front_wheel" params="suffix reflectx reflecty flip" >
-    <joint name="wheel${suffix}" type="continuous" >
-      <parent link="steer${suffix}" />
-      <child link="wheel${suffix}" />
-      <origin xyz="0 0 0" rpy="${-M_PI/2} 0 0" />
-      <axis xyz="0 0 1" />
-    </joint>
-    <link name="wheel${suffix}" >
-      <visual>
-        <origin xyz="0 0.002 0" rpy="0 ${-M_PI/2 + flip*M_PI} 0"/>
-        <geometry>
-          <mesh filename="package://dbw_mkz_description/meshes/wheel.dae" scale="1 1 1" />
-        </geometry>
-      </visual>
-    </link>
-  </xacro:macro>
-  <xacro:macro name="rear_wheel" params="suffix reflectx reflecty flip" >
-    <joint name="wheel${suffix}" type="continuous" >
-      <parent link="base_link" />
-      <child link="wheel${suffix}" />
-      <origin xyz="${reflectx*wheel_base_x} ${reflecty*wheel_base_y} 0" rpy="${-M_PI/2} 0 0" />
-      <axis xyz="0 0 1" />
-    </joint>
-    <link name="wheel${suffix}" >
-      <visual>
-        <origin xyz="0 0.002 0" rpy="0 ${-M_PI/2 + flip*M_PI} 0"/>
-        <geometry>
-          <mesh filename="package://dbw_mkz_description/meshes/wheel.dae" scale="1 1 1" />
-        </geometry>
-      </visual>
-    </link>
-  </xacro:macro>
-  <!-- Base Footprint -->
-  <link name="base_footprint" />
-  <!-- Base Link -->
-  <joint name="footprint" type="fixed" >
-   <parent link="base_footprint" />
-    <child link="base_link" />
-    <origin xyz="0 0 ${wheel_radius+0.09}" rpy="0 0 0" />
-  </joint>
-  <link name="base_link" >
-    <visual>
-      <origin xyz="0 0 -0.3323" rpy="0 0 ${M_PI/2}" />
-      <geometry>
-        <mesh filename="package://dbw_mkz_description/meshes/body.dae" />
-      </geometry>
-    </visual>
-  </link>
-  <xacro:front_wheel suffix="_fl" reflectx=" 1" reflecty=" 1" flip="0" />
-  <xacro:front_wheel suffix="_fr" reflectx=" 1" reflecty=" -1" flip="1" />
-  <xacro:rear_wheel suffix="_rl" reflectx=" 0" reflecty=" 1" flip="0" />
-  <xacro:rear_wheel suffix="_rr" reflectx=" 0" reflecty=" -1" flip="1" />
-  <xacro:steering suffix="_fl" reflecty=" 1" />
-  <xacro:steering suffix="_fr" reflecty=" -1" />
+<robot name="mkz" xmlns:xacro="http://www.ros.org/wiki/xacro" >
+  <xacro:include filename="$(find dbw_mkz_description)/urdf/mkz_13_structure.urdf.xacro" />
 </robot>
